Commit message: fixed laser scannser

File: src/urdf/tb.urdf (robot description, URDF)
Before this commit: robot myfirst, 6 links, 5 joints
Links:
- added link hokuyo_link, mass 1e-5; collision box size=0.1 0.1 0.1; visual mesh filename=package://rrbot_description/meshes/hokuyo.dae
Joints:
- added joint hokuyo_joint: type fixed, parent base_link, child hokuyo_link, origin xyz=1.1 0 0 rpy=0 0 0, axis 1 0 0

Commit message: mapping succesfull

File: src/urdf/tb.urdf (robot description, URDF)
Before this commit: robot myfirst, 7 links, 6 joints
Links:
- link base_link: geometry collision box size=1 1 1; visual box size=1 1 1
Joints:
- joint hokuyo_joint: origin xyz=1.1 0 0 rpy=0 0 0 -> xyz=0.6 0 0 rpy=0 0 0
- joint left_back_wheel_joint: origin xyz=-1 0.38 -0.5 rpy=0 0 0 -> xyz=-0.5 0.5 -0.5 rpy=0 0 0
- joint left_front_wheel_joint: origin xyz=1 0.38 -0.5 -> xyz=0.5 0.5 -0.5
- joint right_back_wheel_joint: origin xyz=-1 -0.38 -0.5 -> xyz=-0.5 -0.5 -0.5
- joint right_front_wheel_joint: origin xyz=1 -0.38 -0.5 -> xyz=0.5 -0.5 -0.5

Commit message: fixed tf error

File: src/urdf/tb.urdf (robot description, URDF)
Before this commit: robot myfirst, 7 links, 6 joints
Links:
- added link imu_link, mass 1; collision cylinder length=0.1 radius=0.1; visual cylinder length=0.1 radius=0.1
Joints:
- added joint imujoint: type fixed, parent base_link, child imu_link
